File: v3/ring_base3.kicad_sch (KiCad schematic)
At the start: 21 parts, among them J1 Conn_01x01_Pin, J2 Conn_01x01_Pin, SW1 TL1015AF160QG, SW2 TL1015AF160QG, SW3 TL1015AF160QG, U1 AT42QT1011-TSHR, U2 AT42QT1011-TSHR, U3 Xiao

Commit message: a small fix
Parts:
- added D1, D2: LED, LED_SMD:LED_0603_1608Metric_Pad1.05x0.95mm_HandSolder, symbol Device:LED
- added R3, R4: R, Resistor_SMD:R_0402_1005Metric_Pad0.72x0.64mm_HandSolder, symbol Device:R
- added SW3, SW8, SW9: TL1015AF160QG, push3x4.5:SW_F160QG_EWI, symbol push3x4.5:TL1015AF160QG
- gave numbers to parts that had none: 3
- renumbered SW2 to SW4, SW3 to SW5
Connections:
- net GND: now also SW3.2, SW8.2, SW9.2
- net VDD: now also D1.2 (A), D2.2 (A)
- net but1: now also SW3.1
- net but2: now also SW8.1
- net but3: now also SW9.1
- net led1: now reaches U3.4 (D3)
- net led1: now also R4.2
- net led: now reaches U3.6 (D5)
- net led: now also R3.2
- new net: D1.1 (K), R3.1
- new net: D2.1 (K), R4.1
- no-connect marks 8 -> 10
